File: hardware/controller_board/controller_board.sch (KiCad schematic (older format))
At the start: 3 parts

Commit message: basic circut outlined
Parts:
- added C1, C2, C3, C4: C, symbol device:C
- added R1, R2, R3, R4: R, symbol device:R
- gave numbers to parts that had none: 3
Connections:
- net labels added: +5V, SCLK_X, SCLK_Y, SDA_X, SDA_Y, SIGNAL_X, SIGNAL_Y, SYNC_X, SYNC_Y
- wire segments 6 -> 52

Commit message: Working up pinouts
Parts:
- added N1, N2, N3, N4: MLTE-DUAL, symbol local:MLTE-DUAL
Connections:
- wire segments 52 -> 35
Other:
- note added: "SIGNAL_OUT"
Changed lines of the file:
@@
-	1    0    0    -1
-$EndComp
-$Comp
-L local:DAC8560 DAC2
-U 1 1 5A852D2B
-P 4100 3350
-F 0 "DAC2" H 4125 3815 50  0000 C CNN
-F 1 "DAC8560" H 4125 3724 50  0000 C CNN
-F 2 "" V 4700 3300 50  0001 C CNN
-F 3 "" V 4700 3300 50  0001 C CNN
-	1    4100 3350
-	1    0    0    -1
-$EndComp
-$Comp
-L local:DAC8560 DAC1
-U 1 1 5A852D67
-P 4100 2300
-F 0 "DAC1" H 4125 2765 50  0000 C CNN
-F 1 "DAC8560" H 4125 2674 50  0000 C CNN
-F 2 "" V 4700 2250 50  0001 C CNN
-F 3 "" V 4700 2250 50  0001 C CNN
-	1    4100 2300
 	1    0    0    -1
 $EndComp
@@
 	1    0    0    -1
 $EndComp
-Wire Wire Line
-	4500 3500 4500 4150
-Wire Wire Line
-	4500 3400 4600 3400
-Wire Wire Line
-	4600 3400 4600 4150
-Wire Wire Line
-	4500 3300 4700 3300
-Wire Wire Line
-	4700 3300 4700 4150
-Wire Wire Line
-	4500 2450 4500 3100
-Wire Wire Line
-	4500 3100 4800 3100
-Wire Wire Line
-	4800 3100 4800 4150
-Wire Wire Line
-	4500 2350 4600 2350
-Wire Wire Line
-	4600 2350 4600 3000
-Wire Wire Line
-	4600 3000 4900 3000
-Wire Wire Line
-	4900 3000 4900 4150
-Wire Wire Line
-	4500 2250 4700 2250
-Wire Wire Line
-	4700 2250 4700 2700
-Wire Wire Line
-	4700 2900 5000 2900
-Wire Wire Line
-	5000 2900 5000 4150
-Connection ~ 4700 2700
-Wire Wire Line
-	4700 2700 4700 2900
-Text GLabel 4500 4150 3    50   Input ~ 0
+Text GLabel 4500 3500 2    50   Input ~ 0
 SYNC_X
-Text GLabel 4600 4150 3    50   Input ~ 0
+Text GLabel 4500 3400 2    50   Input ~ 0
 SCLK_X
-Text GLabel 4700 4150 3    50   Input ~ 0
+Text GLabel 4500 3300 2    50   Input ~ 0
 SDA_X
-Text GLabel 4800 4150 3    50   Input ~ 0
+Text GLabel 4500 2450 2    50   Input ~ 0
 SYNC_Y
-Text GLabel 4900 4150 3    50   Input ~ 0
+Text GLabel 4500 2350 2    50   Input ~ 0
 SCLK_Y
-Text GLabel 5000 4150 3    50   Input ~ 0
+Text GLabel 4500 2250 2    50   Input ~ 0
 SDA_Y
 Wire Wire Line
@@
 Text GLabel 6900 2700 2    50   Input ~ 0
 SIGNAL_X
+$Comp
+L local:MLTE-DUAL N1
+U 1 1 5A87CE82
+P 10300 800
+F 0 "N1" H 10628 871 50  0000 L CNN
+F 1 "MLTE-DUAL" H 10628 780 50  0000 L CNN
+F 2 "" H 10100 800 50  0001 C CNN
+F 3 "" H 10100 800 50  0001 C CNN
+	1    10300 800
+	1    0    0    -1
+$EndComp
+Text Notes 10150 1050 0    50   ~ 0
+SIGNAL_OUT
+Text GLabel 9900 750  0    50   Input ~ 0
+SIGNAL_Y
+Text GLabel 9900 850  0    50   Input ~ 0
+SIGNAL_X
+$Comp
+L local:MLTE-DUAL N2
+U 1 1 5A87E6C9
+P 10350 2300
+F 0 "N2" H 10678 2371 50  0000 L CNN
+F 1 "MLTE-DUAL" H 10678 2280 50  0000 L CNN
+F 2 "" H 10150 2300 50  0001 C CNN
+F 3 "" H 10150 2300 50  0001 C CNN
+	1    10350 2300
+	1    0    0    -1
+$EndComp
+$Comp
+L local:MLTE-DUAL N3
+U 1 1 5A87E731
+P 10350 2650
+F 0 "N3" H 10678 2721 50  0000 L CNN
+F 1 "MLTE-DUAL" H 10678 2630 50  0000 L CNN
+F 2 "" H 10150 2650 50  0001 C CNN
+F 3 "" H 10150 2650 50  0001 C CNN
+	1    10350 2650
+	1    0    0    -1
+$EndComp
+$Comp
+L local:MLTE-DUAL N4
+U 1 1 5A87E781
+P 10350 3000
+F 0 "N4" H 10678 3071 50  0000 L CNN
+F 1 "MLTE-DUAL" H 10678 2980 50  0000 L CNN
+F 2 "" H 10150 3000 50  0001 C CNN
+F 3 "" H 10150 3000 50  0001 C CNN
+	1    10350 3000
+	1    0    0    -1
+$EndComp
+Text GLabel 9950 2250 0    50   Input ~ 0
+SDA_Y
+Text GLabel 9950 2350 0    50   Input ~ 0
+SCLK_Y
+Text GLabel 9950 2600 0    50   Input ~ 0
+SYNC_Y
+Text GLabel 9950 2700 0    50   Input ~ 0
+SDA_X
+Text GLabel 9950 2950 0    50   Input ~ 0
+SCLK_X
+Text GLabel 9950 3050 0    50   Input ~ 0
+SYNC_X
+$Comp
+L local:DAC8560 DAC1
+U 1 1 5A87F2E5
+P 4100 2300
+F 0 "DAC1" H 4125 2765 50  0000 C CNN
+F 1 "DAC8560" H 4125 2674 50  0000 C CNN
+F 2 "" V 4700 2250 50  0001 C CNN
+F 3 "" V 4700 2250 50  0001 C CNN
+	1    4100 2300
+	1    0    0    -1
+$EndComp
+$Comp
+L local:DAC8560 DAC2
+U 1 1 5A87F33F
+P 4100 3350
+F 0 "DAC2" H 4125 3815 50  0000 C CNN
+F 1 "DAC8560" H 4125 3724 50  0000 C CNN
+F 2 "" V 4700 3300 50  0001 C CNN
+F 3 "" V 4700 3300 50  0001 C CNN
+	1    4100 3350
+	1    0    0    -1
+$EndComp
 $EndSCHEMATC
